File: usbtherm-kicad/usbtherm.kicad_pcb (KiCad board)
At the start: 2 copper layers, 27.9 x 67.3 mm, 18 parts, among them IC1 ATMEGA328-P, P1 USB_A_PLUG, Q1 TMP36, Y1 12 MHz

Commit message: fixed wrong USB plug pin layout, other minor layout improvements, removed redundant include
Parts:
- D1: footprint Resistors_ThroughHole:Resistor_Horizontal_RM7mm -> Diode_DO-35_SOD27_Horizontal_RM7
- D2: footprint Resistors_ThroughHole:Resistor_Horizontal_RM7mm -> Diodes_ThroughHole:Diode_DO-35_SOD27_Horizontal_RM7
- moved D1 0.63 mm to (139.1, 86.4)
- moved D2 0.63 mm to (139.1, 91.4)
Connections:
- P1 pad 6: (no net) -> Net-(P1-Pad6)
Routing:
- net GND: track 121.6 -> 0.00 mm
- net Net-(C1-Pad1): track 15.5 -> 13.8 mm
- net Net-(C3-Pad1): track 92.0 -> 90.5 mm
- net Net-(D2-Pad1): track 31.0 -> 32.3 mm
- net Net-(D1-Pad1): track 31.5 -> 30.7 mm
